File: kicad/HEAR.kicad_sch (KiCad schematic)
At the start: 56 parts, among them J1 PJ341, J12 Euro power header, J13 PJ341, J14 PJ341, J2 PJ341, J3 PJ341, J4 PJ341, J5 Attenuator Jumper 1, J6 Attenuator Jumper 2, U1 TL074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

Commit message: added JLCPCB part numbers
Parts:
- C1, C2: LCSC (none) -> C1868
- C10, C7, C8, C9: LCSC (none) -> C14663
- C5, C6: LCSC (none) -> C45783
- D1, D2: footprint nearness:SOD-123 -> Diode_SMD:D_SOD-323_HandSoldering; LCSC (none) -> C191023
- R1, R17, R20, R3, R5, R7: LCSC (none) -> C23196
- R15, R16, R35, R36: LCSC (none) -> C149504
- R19, R38: LCSC (none) -> C25803
- R21, R22, R23, R24, R27, R28: LCSC (none) -> C25804
- R25, R26: LCSC (none) -> C21190
- R29, R30: LCSC (none) -> C23179
- R33, R34: LCSC (none) -> C17903
- U1: LCSC (none) -> SOIC-14_3.9x8.7x1.27P
- U2: LCSC (none) -> C80100

Commit message: gerbers for v01
Parts:
- U1: LCSC SOIC-14_3.9x8.7x1.27P -> C12594
Changed lines of the file:
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@@
       (effects (font (size 1.27 1.27)) hide)
     )
-    (property "LCSC" "SOIC-14_3.9x8.7x1.27P" (id 4) (at 123.19 39.37 0)
+    (property "LCSC" "C12594" (id 4) (at 123.19 39.37 0)
       (effects (font (size 1.27 1.27)) hide)
     )
@@
       (effects (font (size 1.27 1.27)) hide)
     )
-    (property "LCSC" "SOIC-14_3.9x8.7x1.27P" (id 4) (at 161.29 36.83 0)
+    (property "LCSC" "C12594" (id 4) (at 161.29 36.83 0)
       (effects (font (size 1.27 1.27)) hide)
     )
@@
       (effects (font (size 1.27 1.27)) hide)
     )
-    (property "LCSC" "SOIC-14_3.9x8.7x1.27P" (id 4) (at 123.825 101.6 0)
+    (property "LCSC" "C12594" (id 4) (at 123.825 101.6 0)
       (effects (font (size 1.27 1.27)) hide)
     )
@@
       (effects (font (size 1.27 1.27)) hide)
     )
-    (property "LCSC" "SOIC-14_3.9x8.7x1.27P" (id 4) (at 167.005 104.14 0)
+    (property "LCSC" "C12594" (id 4) (at 167.005 104.14 0)
       (effects (font (size 1.27 1.27)) hide)
     )
@@
       (effects (font (size 1.27 1.27)) hide)
     )
-    (property "LCSC" "SOIC-14_3.9x8.7x1.27P" (id 4) (at 247.015 86.995 0)
-      (effects (font (size 1.27 1.27)) hide)
-    )
+    (property "LCSC" "C12594" (id 4) (at 247.015 86.995 0)
+      (effects (font (size 1.27 1.27)) hide)
+    )

Commit message: footprints submodule
Parts:
- J1, J13, J14, J2, J3, J4: footprint nearness:PJ341 -> Crows:PJ341
- RV1: footprint Potentiometer_THT:Potentiometer_Alpha_RD902F-40-00D_Dual_Vertical -> Crows:RV1666G-F
- RV2, RV3, RV4, RV5, RV6, RV7, RV8, RV9: footprint Potentiometer_THT:Potentiometer_Alps_RK09K_Single_Vertical -> Crows:RotaryPotVerticalSingle9mm
Changed lines of the file:
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@@
       (effects (font (size 1.27 1.27)) (justify right))
     )
-    (property "Footprint" "Potentiometer_THT:Potentiometer_Alps_RK09K_Single_Vertical" (id 2) (at 41.275 48.26 0)
+    (property "Footprint" "Crows:RotaryPotVerticalSingle9mm" (id 2) (at 41.275 48.26 0)
       (effects (font (size 1.27 1.27)) hide)
     )
@@
       (effects (font (size 1.27 1.27)) (justify right))
     )
-    (property "Footprint" "Potentiometer_THT:Potentiometer_Alps_RK09K_Single_Vertical" (id 2) (at 41.275 29.845 0)
+    (property "Footprint" "Crows:RotaryPotVerticalSingle9mm" (id 2) (at 41.275 29.845 0)
       (effects (font (size 1.27 1.27)) hide)
     )
@@
       (effects (font (size 1.27 1.27)) (justify right))
     )
-    (property "Footprint" "Potentiometer_THT:Potentiometer_Alps_RK09K_Single_Vertical" (id 2) (at 56.515 29.845 0)
+    (property "Footprint" "Crows:RotaryPotVerticalSingle9mm" (id 2) (at 56.515 29.845 0)
       (effects (font (size 1.27 1.27)) hide)
     )
@@
       (effects (font (size 1.524 1.524)))
     )
-    (property "Footprint" "nearness:PJ341" (id 2) (at 28.575 65.405 0)
+    (property "Footprint" "Crows:PJ341" (id 2) (at 28.575 65.405 0)
       (effects (font (size 1.27 1.27)) hide)
     )
@@
       (effects (font (size 1.524 1.524)))
     )
-    (property "Footprint" "nearness:PJ341" (id 2) (at 28.575 29.845 0)
+    (property "Footprint" "Crows:PJ341" (id 2) (at 28.575 29.845 0)
       (effects (font (size 1.27 1.27)) hide)
     )
@@
       (effects (font (size 1.27 1.27)) (justify right))
     )
-    (property "Footprint" "Potentiometer_THT:Potentiometer_Alps_RK09K_Single_Vertical" (id 2) (at 41.275 83.185 0)
+    (property "Footprint" "Crows:RotaryPotVerticalSingle9mm" (id 2) (at 41.275 83.185 0)
       (effects (font (size 1.27 1.27)) hide)
     )
@@
       (effects (font (size 1.27 1.27)) (justify right))
     )
-    (property "Footprint" "Potentiometer_THT:Potentiometer_Alps_RK09K_Single_Vertical" (id 2) (at 41.275 65.405 0)
+    (property "Footprint" "Crows:RotaryPotVerticalSingle9mm" (id 2) (at 41.275 65.405 0)
       (effects (font (size 1.27 1.27)) hide)
     )
@@
       (effects (font (size 1.524 1.524)))
     )
-    (property "Footprint" "nearness:PJ341" (id 2) (at 28.575 48.26 0)
+    (property "Footprint" "Crows:PJ341" (id 2) (at 28.575 48.26 0)
       (effects (font (size 1.27 1.27)) hide)
     )
@@
       (effects (font (size 1.27 1.27)) (justify right))
     )
-    (property "Footprint" "Potentiometer_THT:Potentiometer_Alps_RK09K_Single_Vertical" (id 2) (at 56.515 48.26 0)
+    (property "Footprint" "Crows:RotaryPotVerticalSingle9mm" (id 2) (at 56.515 48.26 0)
       (effects (font (size 1.27 1.27)) hide)
     )
@@
       (effects (font (size 1.524 1.524)))
     )
-    (property "Footprint" "nearness:PJ341" (id 2) (at 242.57 126.492 0)
+    (property "Footprint" "Crows:PJ341" (id 2) (at 242.57 126.492 0)
       (effects (font (size 1.27 1.27)) hide)
     )
@@
       (effects (font (size 1.27 1.27)) (justify right) hide)
     )
-    (property "Footprint" "Potentiometer_THT:Potentiometer_Alpha_RD902F-40-00D_Dual_Vertical" (id 2) (at 80.645 167.64 0)
+    (property "Footprint" "Crows:RV1666G-F" (id 2) (at 80.645 167.64 0)
       (effects (font (size 1.27 1.27)) hide)
     )
@@
       (effects (font (size 1.27 1.27)) (justify right) hide)
     )
-    (property "Footprint" "Potentiometer_THT:Potentiometer_Alpha_RD902F-40-00D_Dual_Vertical" (id 2) (at 80.645 131.445 0)
+    (property "Footprint" "Crows:RV1666G-F" (id 2) (at 80.645 131.445 0)
       (effects (font (size 1.27 1.27)) hide)
     )
@@
       (effects (font (size 1.524 1.524)))
     )
-    (property "Footprint" "nearness:PJ341" (id 2) (at 28.575 83.185 0)
+    (property "Footprint" "Crows:PJ341" (id 2) (at 28.575 83.185 0)
       (effects (font (size 1.27 1.27)) hide)
     )
@@
       (effects (font (size 1.27 1.27)) (justify right))
     )
-    (property "Footprint" "Potentiometer_THT:Potentiometer_Alps_RK09K_Single_Vertical" (id 2) (at 56.515 65.405 0)
+    (property "Footprint" "Crows:RotaryPotVerticalSingle9mm" (id 2) (at 56.515 65.405 0)
       (effects (font (size 1.27 1.27)) hide)
     )
@@
       (effects (font (size 1.27 1.27)) (justify right))
     )
-    (property "Footprint" "Potentiometer_THT:Potentiometer_Alps_RK09K_Single_Vertical" (id 2) (at 56.515 83.185 0)
+    (property "Footprint" "Crows:RotaryPotVerticalSingle9mm" (id 2) (at 56.515 83.185 0)
       (effects (font (size 1.27 1.27)) hide)
     )
@@
       (effects (font (size 1.524 1.524)))
     )
-    (property "Footprint" "nearness:PJ341" (id 2) (at 242.57 148.336 0)
+    (property "Footprint" "Crows:PJ341" (id 2) (at 242.57 148.336 0)
       (effects (font (size 1.27 1.27)) hide)
     )
@@
     )
     (path "/2d1ad5ac-7622-48a8-a54c-7612daf81ae4"
-      (reference "J1") (unit 1) (value "PJ341") (footprint "nearness:PJ341")
+      (reference "J1") (unit 1) (value "PJ341") (footprint "Crows:PJ341")
     )
     (path "/65aa5a5e-a3f2-4489-b0b5-85e25933a0f6"
-      (reference "J2") (unit 1) (value "PJ341") (footprint "nearness:PJ341")
+      (reference "J2") (unit 1) (value "PJ341") (footprint "Crows:PJ341")
     )
     (path "/22ec142d-dd8e-422e-9e28-8e29da427d0b"
-      (reference "J3") (unit 1) (value "PJ341") (footprint "nearness:PJ341")
+      (reference "J3") (unit 1) (value "PJ341") (footprint "Crows:PJ341")
     )
     (path "/92418c4a-8bde-4fc6-bdda-b669335ef2b0"
-      (reference "J4") (unit 1) (value "PJ341") (footprint "nearness:PJ341")
+      (reference "J4") (unit 1) (value "PJ341") (footprint "Crows:PJ341")
     )
     (path "/a7e7f0c0-b9cf-4531-8150-823ec51bef19"
@@
     )
     (path "/6ad14557-273d-4afc-aa78-30c3e4670cc4"
-      (reference "J13") (unit 1) (value "PJ341") (footprint "nearness:PJ341")
+      (reference "J13") (unit 1) (value "PJ341") (footprint "Crows:PJ341")
     )
     (path "/ed608030-d287-4d9a-b3c0-106d7268fec2"
-      (reference "J14") (unit 1) (value "PJ341") (footprint "nearness:PJ341")
+      (reference "J14") (unit 1) (value "PJ341") (footprint "Crows:PJ341")
     )
     (path "/2b498836-838b-4c57-8fb4-88dbab659fbd"
@@
     )
     (path "/7114b75a-5eeb-4616-96ea-dfea1d42f03c"
-      (reference "RV1") (unit 1) (value "B10K") (footprint "Potentiometer_THT:Potentiometer_Alpha_RD902F-40-00D_Dual_Vertical")
+      (reference "RV1") (unit 1) (value "B10K") (footprint "Crows:RV1666G-F")
     )
     (path "/6e9bf8f1-f262-4b27-b3ad-c125c7a9d14a"
-      (reference "RV1") (unit 2) (value "B10K") (footprint "Potentiometer_THT:Potentiometer_Alpha_RD902F-40-00D_Dual_Vertical")
+      (reference "RV1") (unit 2) (value "B10K") (footprint "Crows:RV1666G-F")
     )
     (path "/0ed6a872-6c2d-431f-9e74-9e26ef2d81f2"
-      (reference "RV2") (unit 1) (value "10K Vol") (footprint "Potentiometer_THT:Potentiometer_Alps_RK09K_Single_Vertical")
+      (reference "RV2") (unit 1) (value "10K Vol") (footprint "Crows:RotaryPotVerticalSingle9mm")
     )
     (path "/0812653a-f06a-4bc2-ad1c-93f1009d63a9"
-      (reference "RV3") (unit 1) (value "10K Vol") (footprint "Potentiometer_THT:Potentiometer_Alps_RK09K_Single_Vertical")
+      (reference "RV3") (unit 1) (value "10K Vol") (footprint "Crows:RotaryPotVerticalSingle9mm")
     )
     (path "/54a7fc3f-5b9a-41c8-bcc9-ba0281cbc143"
-      (reference "RV4") (unit 1) (value "10K Vol") (footprint "Potentiometer_THT:Potentiometer_Alps_RK09K_Single_Vertical")
+      (reference "RV4") (unit 1) (value "10K Vol") (footprint "Crows:RotaryPotVerticalSingle9mm")
     )
     (path "/3b1facd0-70b5-4407-8bdd-9315ce97fd11"
-      (reference "RV5") (unit 1) (value "10K Vol") (footprint "Potentiometer_THT:Potentiometer_Alps_RK09K_Single_Vertical")
+      (reference "RV5") (unit 1) (value "10K Vol") (footprint "Crows:RotaryPotVerticalSingle9mm")
     )
     (path "/1fe0a425-49de-41eb-bb4f-73980c154fef"
-      (reference "RV6") (unit 1) (value "10K") (footprint "Potentiometer_THT:Potentiometer_Alps_RK09K_Single_Vertical")
+      (reference "RV6") (unit 1) (value "10K") (footprint "Crows:RotaryPotVerticalSingle9mm")
     )
     (path "/69f1b745-eaf5-4060-a939-51e36ca8d1f3"
-      (reference "RV7") (unit 1) (value "10K") (footprint "Potentiometer_THT:Potentiometer_Alps_RK09K_Single_Vertical")
+      (reference "RV7") (unit 1) (value "10K") (footprint "Crows:RotaryPotVerticalSingle9mm")
     )
     (path "/9c7cb67d-1ebc-4329-98eb-7a7c3f951a41"
-      (reference "RV8") (unit 1) (value "10K") (footprint "Potentiometer_THT:Potentiometer_Alps_RK09K_Single_Vertical")
+      (reference "RV8") (unit 1) (value "10K") (footprint "Crows:RotaryPotVerticalSingle9mm")
     )
     (path "/ad4cd9c4-4679-4c36-bb93-b5b0c1bdbe48"
-      (reference "RV9") (unit 1) (value "10K") (footprint "Potentiometer_THT:Potentiometer_Alps_RK09K_Single_Vertical")
+      (reference "RV9") (unit 1) (value "10K") (footprint "Crows:RotaryPotVerticalSingle9mm")
     )
     (path "/00000000-0000-0000-0000-000059a3b25b"

Commit message: updated library, new footprint names
Parts:
- J1, J13, J14, J2, J3, J4: footprint Crows:PJ341 -> Crows:PJ341_3.5mm_headphone
- RV2, RV3, RV4, RV5, RV6, RV7, RV8, RV9: footprint Crows:RotaryPotVerticalSingle9mm -> Crows:Potentiometer_Rotary_9mm_Vertical_Single
Changed lines of the file:
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@@
       (effects (font (size 1.27 1.27)) (justify right))
     )
-    (property "Footprint" "Crows:RotaryPotVerticalSingle9mm" (id 2) (at 41.275 48.26 0)
+    (property "Footprint" "Crows:Potentiometer_Rotary_9mm_Vertical_Single" (id 2) (at 41.275 48.26 0)
       (effects (font (size 1.27 1.27)) hide)
     )
@@
       (effects (font (size 1.27 1.27)) (justify right))
     )
-    (property "Footprint" "Crows:RotaryPotVerticalSingle9mm" (id 2) (at 41.275 29.845 0)
+    (property "Footprint" "Crows:Potentiometer_Rotary_9mm_Vertical_Single" (id 2) (at 41.275 29.845 0)
       (effects (font (size 1.27 1.27)) hide)
     )
@@
       (effects (font (size 1.27 1.27)) (justify right))
     )
-    (property "Footprint" "Crows:RotaryPotVerticalSingle9mm" (id 2) (at 56.515 29.845 0)
+    (property "Footprint" "Crows:Potentiometer_Rotary_9mm_Vertical_Single" (id 2) (at 56.515 29.845 0)
       (effects (font (size 1.27 1.27)) hide)
     )
@@
       (effects (font (size 1.524 1.524)))
     )
-    (property "Footprint" "Crows:PJ341" (id 2) (at 28.575 65.405 0)
+    (property "Footprint" "Crows:PJ341_3.5mm_headphone" (id 2) (at 28.575 65.405 0)
       (effects (font (size 1.27 1.27)) hide)
     )
@@
       (effects (font (size 1.524 1.524)))
     )
-    (property "Footprint" "Crows:PJ341" (id 2) (at 28.575 29.845 0)
+    (property "Footprint" "Crows:PJ341_3.5mm_headphone" (id 2) (at 28.575 29.845 0)
       (effects (font (size 1.27 1.27)) hide)
     )
@@
       (effects (font (size 1.27 1.27)) (justify right))
     )
-    (property "Footprint" "Crows:RotaryPotVerticalSingle9mm" (id 2) (at 41.275 83.185 0)
+    (property "Footprint" "Crows:Potentiometer_Rotary_9mm_Vertical_Single" (id 2) (at 41.275 83.185 0)
       (effects (font (size 1.27 1.27)) hide)
     )
@@
       (effects (font (size 1.27 1.27)) (justify right))
     )
-    (property "Footprint" "Crows:RotaryPotVerticalSingle9mm" (id 2) (at 41.275 65.405 0)
+    (property "Footprint" "Crows:Potentiometer_Rotary_9mm_Vertical_Single" (id 2) (at 41.275 65.405 0)
       (effects (font (size 1.27 1.27)) hide)
     )
@@
       (effects (font (size 1.524 1.524)))
     )
-    (property "Footprint" "Crows:PJ341" (id 2) (at 28.575 48.26 0)
+    (property "Footprint" "Crows:PJ341_3.5mm_headphone" (id 2) (at 28.575 48.26 0)
       (effects (font (size 1.27 1.27)) hide)
     )
@@
       (effects (font (size 1.27 1.27)) (justify right))
     )
-    (property "Footprint" "Crows:RotaryPotVerticalSingle9mm" (id 2) (at 56.515 48.26 0)
+    (property "Footprint" "Crows:Potentiometer_Rotary_9mm_Vertical_Single" (id 2) (at 56.515 48.26 0)
       (effects (font (size 1.27 1.27)) hide)
     )
@@
       (effects (font (size 1.524 1.524)))
     )
-    (property "Footprint" "Crows:PJ341" (id 2) (at 242.57 126.492 0)
+    (property "Footprint" "Crows:PJ341_3.5mm_headphone" (id 2) (at 242.57 126.492 0)
       (effects (font (size 1.27 1.27)) hide)
     )
@@
       (effects (font (size 1.524 1.524)))
     )
-    (property "Footprint" "Crows:PJ341" (id 2) (at 28.575 83.185 0)
+    (property "Footprint" "Crows:PJ341_3.5mm_headphone" (id 2) (at 28.575 83.185 0)
       (effects (font (size 1.27 1.27)) hide)
     )
@@
       (effects (font (size 1.27 1.27)) (justify right))
     )
-    (property "Footprint" "Crows:RotaryPotVerticalSingle9mm" (id 2) (at 56.515 65.405 0)
+    (property "Footprint" "Crows:Potentiometer_Rotary_9mm_Vertical_Single" (id 2) (at 56.515 65.405 0)
       (effects (font (size 1.27 1.27)) hide)
     )
@@
       (effects (font (size 1.27 1.27)) (justify right))
     )
-    (property "Footprint" "Crows:RotaryPotVerticalSingle9mm" (id 2) (at 56.515 83.185 0)
+    (property "Footprint" "Crows:Potentiometer_Rotary_9mm_Vertical_Single" (id 2) (at 56.515 83.185 0)
       (effects (font (size 1.27 1.27)) hide)
     )
@@
       (effects (font (size 1.524 1.524)))
     )
-    (property "Footprint" "Crows:PJ341" (id 2) (at 242.57 148.336 0)
+    (property "Footprint" "Crows:PJ341_3.5mm_headphone" (id 2) (at 242.57 148.336 0)
       (effects (font (size 1.27 1.27)) hide)
     )
@@
     )
     (path "/2d1ad5ac-7622-48a8-a54c-7612daf81ae4"
-      (reference "J1") (unit 1) (value "PJ341") (footprint "Crows:PJ341")
+      (reference "J1") (unit 1) (value "PJ341") (footprint "Crows:PJ341_3.5mm_headphone")
     )
     (path "/65aa5a5e-a3f2-4489-b0b5-85e25933a0f6"
-      (reference "J2") (unit 1) (value "PJ341") (footprint "Crows:PJ341")
+      (reference "J2") (unit 1) (value "PJ341") (footprint "Crows:PJ341_3.5mm_headphone")
     )
     (path "/22ec142d-dd8e-422e-9e28-8e29da427d0b"
-      (reference "J3") (unit 1) (value "PJ341") (footprint "Crows:PJ341")
+      (reference "J3") (unit 1) (value "PJ341") (footprint "Crows:PJ341_3.5mm_headphone")
     )
     (path "/92418c4a-8bde-4fc6-bdda-b669335ef2b0"
-      (reference "J4") (unit 1) (value "PJ341") (footprint "Crows:PJ341")
+      (reference "J4") (unit 1) (value "PJ341") (footprint "Crows:PJ341_3.5mm_headphone")
     )
     (path "/a7e7f0c0-b9cf-4531-8150-823ec51bef19"
@@
     )
     (path "/6ad14557-273d-4afc-aa78-30c3e4670cc4"
-      (reference "J13") (unit 1) (value "PJ341") (footprint "Crows:PJ341")
+      (reference "J13") (unit 1) (value "PJ341") (footprint "Crows:PJ341_3.5mm_headphone")
     )
     (path "/ed608030-d287-4d9a-b3c0-106d7268fec2"
-      (reference "J14") (unit 1) (value "PJ341") (footprint "Crows:PJ341")
+      (reference "J14") (unit 1) (value "PJ341") (footprint "Crows:PJ341_3.5mm_headphone")
     )
     (path "/2b498836-838b-4c57-8fb4-88dbab659fbd"
@@
     )
     (path "/0ed6a872-6c2d-431f-9e74-9e26ef2d81f2"
-      (reference "RV2") (unit 1) (value "10K Vol") (footprint "Crows:RotaryPotVerticalSingle9mm")
+      (reference "RV2") (unit 1) (value "10K Vol") (footprint "Crows:Potentiometer_Rotary_9mm_Vertical_Single")
     )
     (path "/0812653a-f06a-4bc2-ad1c-93f1009d63a9"
-      (reference "RV3") (unit 1) (value "10K Vol") (footprint "Crows:RotaryPotVerticalSingle9mm")
+      (reference "RV3") (unit 1) (value "10K Vol") (footprint "Crows:Potentiometer_Rotary_9mm_Vertical_Single")
     )
     (path "/54a7fc3f-5b9a-41c8-bcc9-ba0281cbc143"
-      (reference "RV4") (unit 1) (value "10K Vol") (footprint "Crows:RotaryPotVerticalSingle9mm")
+      (reference "RV4") (unit 1) (value "10K Vol") (footprint "Crows:Potentiometer_Rotary_9mm_Vertical_Single")
     )
     (path "/3b1facd0-70b5-4407-8bdd-9315ce97fd11"
-      (reference "RV5") (unit 1) (value "10K Vol") (footprint "Crows:RotaryPotVerticalSingle9mm")
+      (reference "RV5") (unit 1) (value "10K Vol") (footprint "Crows:Potentiometer_Rotary_9mm_Vertical_Single")
     )
     (path "/1fe0a425-49de-41eb-bb4f-73980c154fef"
-      (reference "RV6") (unit 1) (value "10K") (footprint "Crows:RotaryPotVerticalSingle9mm")
+      (reference "RV6") (unit 1) (value "10K") (footprint "Crows:Potentiometer_Rotary_9mm_Vertical_Single")
     )
     (path "/69f1b745-eaf5-4060-a939-51e36ca8d1f3"
-      (reference "RV7") (unit 1) (value "10K") (footprint "Crows:RotaryPotVerticalSingle9mm")
+      (reference "RV7") (unit 1) (value "10K") (footprint "Crows:Potentiometer_Rotary_9mm_Vertical_Single")
     )
     (path "/9c7cb67d-1ebc-4329-98eb-7a7c3f951a41"
-      (reference "RV8") (unit 1) (value "10K") (footprint "Crows:RotaryPotVerticalSingle9mm")
+      (reference "RV8") (unit 1) (value "10K") (footprint "Crows:Potentiometer_Rotary_9mm_Vertical_Single")
     )
     (path "/ad4cd9c4-4679-4c36-bb93-b5b0c1bdbe48"
-      (reference "RV9") (unit 1) (value "10K") (footprint "Crows:RotaryPotVerticalSingle9mm")
+      (reference "RV9") (unit 1) (value "10K") (footprint "Crows:Potentiometer_Rotary_9mm_Vertical_Single")
     )
     (path "/00000000-0000-0000-0000-000059a3b25b"

Commit message: v3 gerbers (had to swap out a cap, part no longer available
Parts:
- C5, C6: footprint Capacitor_SMD:C_0805_2012Metric_Pad1.18x1.45mm_HandSolder -> Capacitor_SMD:C_1206_3216Metric_Pad1.33x1.80mm_HandSolder; LCSC C45783 -> C12891
Changed lines of the file:
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@@
       (effects (font (size 1.27 1.27)) (justify left))
     )
-    (property "Footprint" "Capacitor_SMD:C_0805_2012Metric_Pad1.18x1.45mm_HandSolder" (id 2) (at 242.0112 35.814 0)
+    (property "Footprint" "Capacitor_SMD:C_1206_3216Metric_Pad1.33x1.80mm_HandSolder" (id 2) (at 242.0112 35.814 0)
       (effects (font (size 1.27 1.27)) hide)
     )
     (property "Datasheet" "" (id 3) (at 241.046 32.004 0))
-    (property "LCSC" "C45783" (id 4) (at 241.046 32.004 0)
+    (property "LCSC" "C12891" (id 4) (at 241.046 32.004 0)
       (effects (font (size 1.27 1.27)) hide)
     )
@@
       (effects (font (size 1.27 1.27)) (justify left))
     )
-    (property "Footprint" "Capacitor_SMD:C_0805_2012Metric_Pad1.18x1.45mm_HandSolder" (id 2) (at 242.0112 48.514 0)
+    (property "Footprint" "Capacitor_SMD:C_1206_3216Metric_Pad1.33x1.80mm_HandSolder" (id 2) (at 242.0112 48.514 0)
       (effects (font (size 1.27 1.27)) hide)
     )
     (property "Datasheet" "" (id 3) (at 241.046 44.704 0))
-    (property "LCSC" "C45783" (id 4) (at 241.046 44.704 0)
+    (property "LCSC" "C12891" (id 4) (at 241.046 44.704 0)
       (effects (font (size 1.27 1.27)) hide)
     )
@@
     )
     (path "/00000000-0000-0000-0000-000058fd9a5f"
-      (reference "C5") (unit 1) (value "22u") (footprint "Capacitor_SMD:C_0805_2012Metric_Pad1.18x1.45mm_HandSolder")
+      (reference "C5") (unit 1) (value "22u") (footprint "Capacitor_SMD:C_1206_3216Metric_Pad1.33x1.80mm_HandSolder")
     )
     (path "/00000000-0000-0000-0000-000058fd9b16"
-      (reference "C6") (unit 1) (value "22u") (footprint "Capacitor_SMD:C_0805_2012Metric_Pad1.18x1.45mm_HandSolder")
+      (reference "C6") (unit 1) (value "22u") (footprint "Capacitor_SMD:C_1206_3216Metric_Pad1.33x1.80mm_HandSolder")
     )
     (path "/00000000-0000-0000-0000-000058fd9c65"
